File: electrical/panel.kicad_sch (KiCad schematic)
At the start: 1 part

Commit message: 🎮 Working on electrical schematic
Parts:
- removed U11: ~, symbol Garmin:GAD27
Other:
- added sheet Power (power.kicad_sch)
- added sheet Sensors (sensors.kicad_sch)
