File: electrical/fuse_central.kicad_sch (KiCad schematic)
At the start: 1 part, among them U5 ROLL TRIM

Commit message: 🎮 Working on electrical schematic
Parts:
- renumbered U5 to C1
Connections:
- net ROLL.SENSE renamed ROLL_TRIM_POS
- net ROLL.SENSE_HI renamed ROLL_TRIM_POS_HI
- net ROLL.SENSE_LO renamed ROLL_TRIM_POS_LO
- net ROLL_TRIM.TRIM1 renamed ROLL_AP_TRIM1
- net ROLL_TRIM.TRIM2 renamed ROLL_AP_TRIM2
Other:
- moved on the sheet: C1

Commit message: 📆 Weekend work
Changed lines of the file:
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@@
+	)
+	(bus_entry
+		(at 34.29 49.53)
+		(size 2.54 -2.54)
+		(stroke
+			(width 0)
+			(type default)
+		)
 	)
 	(bus_entry
@@
 	)
 	(bus_entry
+		(at 95.25 44.45)
+		(size 2.54 2.54)
+		(stroke
+			(width 0)
+			(type default)
+		)
+	)
+	(bus_entry
 		(at 53.34 90.17)
 		(size 2.54 2.54)
@@
 	)
 	(bus_entry
+		(at 95.25 46.99)
+		(size 2.54 2.54)
+		(stroke
+			(width 0)
+			(type default)
+		)
+	)
+	(bus_entry
 		(at 181.61 151.13)
 		(size -2.54 2.54)
@@
 	)
 	(bus_entry
+		(at 34.29 46.99)
+		(size 2.54 -2.54)
+		(stroke
+			(width 0)
+			(type default)
+		)
+	)
+	(bus_entry
 		(at 100.33 36.83)
 		(size -2.54 2.54)
@@
 	(wire
 		(pts
+			(xy 36.83 44.45) (xy 95.25 44.45)
+		)
+		(stroke
+			(width 0)
+			(type default)
+		)
+	)
+	(wire
+		(pts
 			(xy 58.42 85.09) (xy 95.25 85.09)
 		)
@@
 		)
 	)
+	(wire
+		(pts
+			(xy 36.83 46.99) (xy 95.25 46.99)
+		)
+		(stroke
+			(width 0)
+			(type default)
+		)
+	)
 	(bus
 		(pts
@@
 	(bus
 		(pts
-			(xy 97.79 44.45) (xy 97.79 64.77)
+			(xy 97.79 44.45) (xy 97.79 46.99)
 		)
 		(stroke
@@
 	(bus
 		(pts
-			(xy 34.29 44.45) (xy 34.29 67.31)
+			(xy 34.29 44.45) (xy 34.29 46.99)
+		)
+		(stroke
+			(width 0)
+			(type default)
+		)
+	)
+	(bus
+		(pts
+			(xy 97.79 49.53) (xy 97.79 64.77)
 		)
 		(stroke
@@
 		)
 	)
+	(bus
+		(pts
+			(xy 34.29 46.99) (xy 34.29 49.53)
+		)
+		(stroke
+			(width 0)
+			(type default)
+		)
+	)
 	(wire
 		(pts
@@
 		)
 	)
+	(bus
+		(pts
+			(xy 34.29 49.53) (xy 34.29 67.31)
+		)
+		(stroke
+			(width 0)
+			(type default)
+		)
+	)
 	(wire
 		(pts
@@
 		(pts
 			(xy 100.33 41.91) (xy 179.07 41.91)
+		)
+		(stroke
+			(width 0)
+			(type default)
+		)
+	)
+	(bus
+		(pts
+			(xy 97.79 46.99) (xy 97.79 49.53)
 		)
 		(stroke
@@
 		)
 	)
+	(label "PITOT_TEMP"
+		(at 58.42 46.99 0)
+		(effects
+			(font
+				(size 1.27 1.27)
+			)
+			(justify left bottom)
+		)
+	)
 	(label "ROLL_AP_12V"
 		(at 123.19 62.23 0)
@@
 		(effects
 			(font
+				(size 1.27 1.27)
+			)
+			(justify left bottom)
+		)
+	)
+	(label "STALL_SENSOR"
+		(at 58.42 44.45 0)
+		(effects
+			(font
