File: electrical/sensors.kicad_sch (KiCad schematic)
At the start: 3 parts, among them U4 GAD27 J271, U5 GAD27 J272, U6 GAD27 TB273

Commit message: 📆 Weekend work
Parts:
- added U7: ~, symbol Garmin:GEA24_J244
Connections:
- new net PITOT_TEMP: U7.41 (DISCRETE_IN2)
- new net STALL_SENSOR: U7.40 (DISCRETE_IN1)
