File: electrical/wing_left.kicad_sch (KiCad schematic)
At the start: 5 parts

Commit message: 🎮 Working on electrical schematic
Connections:
- net GND: now also LW3.2 (GND); no longer LW3. (GND)
- removed net FUEL: LW3. (GND)
- net LANDING_12V renamed LEFT_LAND
- net LIGHT.POSN+ renamed LEFT_POSN+
- net LIGHT.POSN- renamed LEFT_POSN-
- net LIGHT.STROBE+ renamed LEFT_STROBE+
- net LIGHT.STROBE- renamed LEFT_STROBE-
- net TAXI renamed LEFT_TAXI
- new net LEFT_FUEL: LW3.1 (QTY)
Other:
- moved on the sheet: LW4, LW5

Commit message: 📆 Weekend work
Parts:
- added LW5: STALL SENSOR, symbol Misc:SWITCH
- renumbered LW5 to LW6
Connections:
- net GND: now also LW5.1
- new net STALL_SENSOR: LW5.2
Other:
- moved on the sheet: LW6
Changed lines of the file:
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@@
+	)
+	(bus_entry
+		(at 96.52 137.16)
+		(size -2.54 2.54)
+		(stroke
+			(width 0)
+			(type default)
+		)
 	)
 	(bus_entry
@@
 	)
 	(bus_entry
-		(at 96.52 135.89)
+		(at 96.52 168.91)
 		(size -2.54 2.54)
 		(stroke
@@
 	(wire
 		(pts
+			(xy 40.64 139.7) (xy 40.64 143.51)
+		)
+		(stroke
+			(width 0)
+			(type default)
+		)
+	)
+	(wire
+		(pts
 			(xy 67.31 91.44) (xy 67.31 93.98)
 		)
@@
 	(wire
 		(pts
+			(xy 60.96 139.7) (xy 93.98 139.7)
+		)
+		(stroke
+			(width 0)
+			(type default)
+		)
+	)
+	(wire
+		(pts
 			(xy 39.37 114.3) (xy 39.37 116.84)
 		)
@@
 	(wire
 		(pts
-			(xy 50.8 138.43) (xy 93.98 138.43)
-		)
-		(stroke
-			(width 0)
-			(type default)
-		)
-	)
-	(wire
-		(pts
-			(xy 50.8 138.43) (xy 50.8 134.62)
+			(xy 50.8 171.45) (xy 93.98 171.45)
+		)
+		(stroke
+			(width 0)
+			(type default)
+		)
+	)
+	(wire
+		(pts
+			(xy 50.8 171.45) (xy 50.8 167.64)
 		)
 		(stroke
@@
 		)
 	)
+	(bus
+		(pts
+			(xy 96.52 137.16) (xy 96.52 168.91)
+		)
+		(stroke
+			(width 0)
+			(type default)
+		)
+	)
 	(wire
 		(pts
@@
 	(bus
 		(pts
-			(xy 96.52 110.49) (xy 96.52 135.89)
+			(xy 96.52 110.49) (xy 96.52 137.16)
 		)
 		(stroke
@@
 		(pts
 			(xy 91.44 33.02) (xy 91.44 46.99)
+		)
+		(stroke
+			(width 0)
+			(type default)
+		)
+	)
+	(wire
+		(pts
+			(xy 45.72 139.7) (xy 40.64 139.7)
 		)
 		(stroke
@@
 		)
 	)
+	(label "STALL_SENSOR"
+		(at 80.01 139.7 0)
+		(effects
+			(font
+				(size 1.27 1.27)
+			)
+			(justify left bottom)
+		)
+	)
 	(label "LEFT_LAND"
 		(at 82.55 71.12 0)
@@
 	)
 	(label "NAV"
-		(at 90.17 138.43 0)
+		(at 90.17 171.45 0)
 		(effects
 			(font
@@
 	(symbol
 		(lib_id "Misc:ANTENNA")
-		(at 50.8 128.27 0)
+		(at 50.8 161.29 0)
 		(unit 1)
 		(exclude_from_sim no)
@@
 		(dnp no)
 		(fields_autoplaced yes)
-		(property "Reference" "LW5"
-			(at 50.165 124.46 0)
-			(effects
-				(font
-					(size 1.27 1.27)
-				)
+		(property "Reference" "LW6"
+			(at 53.34 163.1949 0)
+			(effects
+				(font
+					(size 1.27 1.27)
+				)
+				(justify left)
 			)
 		)
 		(property "Value" "ARCHER MODEL 1 LEFT"
-			(at 50.165 127 0)
-			(effects
-				(font
-					(size 1.27 1.27)
-				)
+			(at 53.34 165.7349 0)
+			(effects
+				(font
+					(size 1.27 1.27)
+				)
+				(justify left)
 			)
 		)
 		(property "Footprint" ""
-			(at 50.8 128.27 0)
+			(at 50.8 161.29 0)
 			(effects
 				(font
@@
 		)
 		(property "Datasheet" ""
-			(at 50.8 128.27 0)
+			(at 50.8 161.29 0)
 			(effects
 				(font
@@
 		)
 		(property "Description" ""
-			(at 50.8 128.27 0)
+			(at 50.8 161.29 0)
 			(effects
 				(font
@@
 			(project ""
 				(path "/8f70a519-989e-4461-b188-ee220b2df3e4/e072061e-a93d-46df-af9c-1a54acb5961b"
-					(reference "LW5")
+					(reference "LW6")
 					(unit 1)
 				)
@@
 					(unit 1)
 				)
+			)
+		)
+	)
+	(symbol
+		(lib_id "Misc:SWITCH")
+		(at 53.34 135.89 0)
+		(unit 1)
+		(exclude_from_sim no)
+		(in_bom yes)
+		(on_board yes)
+		(dnp no)
+		(fields_autoplaced yes)
+		(property "Reference" "LW5"
+			(at 53.34 132.08 0)
+			(effects
+				(font
+					(size 1.27 1.27)
+				)
+			)
+		)
+		(property "Value" "STALL SENSOR"
+			(at 53.34 134.62 0)
+			(effects
+				(font
+					(size 1.27 1.27)
+				)
+			)
+		)
+		(property "Footprint" ""
+			(at 53.34 135.89 0)
+			(effects
+				(font
+					(size 1.27 1.27)
+				)
+				(hide yes)
+			)
+		)
+		(property "Datasheet" ""
+			(at 53.34 135.89 0)
+			(effects
+				(font
+					(size 1.27 1.27)
+				)
+				(hide yes)
+			)
+		)
+		(property "Description" ""
+			(at 53.34 135.89 0)
+			(effects
+				(font
+					(size 1.27 1.27)
+				)
+				(hide yes)
+			)
+		)
+		(pin "1"
+		)
+		(pin "2"
+		)
+		(instances
+			(project ""
+				(path "/8f70a519-989e-4461-b188-ee220b2df3e4/e072061e-a93d-46df-af9c-1a54acb5961b"
+					(reference "LW5")
+					(unit 1)
+				)
+			)
+		)
+	)
+	(symbol
+		(lib_id "Misc:GND")
+		(at 40.64 144.78 0)
+		(unit 1)
+		(exclude_from_sim no)
+		(in_bom yes)
+		(on_board yes)
+		(dnp no)
+		(fields_autoplaced yes)
+		(property "Reference" "#PWR016"
+			(at 37.846 139.192 0)
+			(effects
+				(font
+					(size 1.27 1.27)
+				)
+				(hide yes)
+			)
+		)
+		(property "Value" "GND"
+			(at 40.64 144.78 0)
+			(effects
+				(font
+					(size 1.27 1.27)
+				)
+				(hide yes)
+			)
+		)
+		(property "Footprint" ""
+			(at 40.64 144.78 0)
+			(effects
+				(font
+					(size 1.27 1.27)
+				)
+				(hide yes)
+			)
+		)
+		(property "Datasheet" ""
+			(at 40.64 144.78 0)
+			(effects
+				(font
+					(size 1.27 1.27)
+				)
+				(hide yes)
+			)
+		)
+		(property "Description" ""
+			(at 40.64 144.78 0)
+			(effects
+				(font
+					(size 1.27 1.27)
+				)
+				(hide yes)
+			)
+		)
+		(pin "1"
+		)
+		(instances
+			(project "electrical"
+				(path "/8f70a519-989e-4461-b188-ee220b2df3e4/e072061e-a93d-46df-af9c-1a54acb5961b"
+					(reference "#PWR016")
+					(unit 1)
+				)
